File: pcb/piconsole.kicad_pcb (KiCad board)
At the start: 2 copper layers, 67.3 x 80.6 mm, 28 parts, among them J1 Bat, J2 GPIO, SW1 Up, SW2 Down, SW3 Left, SW4 Right, SW5 A, SW6 B, SW7 SW_SPDT, SW8 RESET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

Commit message: v7. Enrutado más directo a LED IR.
Routing:
- net L_IR: track 103.9 -> 81.0 mm, vias 2 -> 1
Other:
- board text added: "niubit PiConsole v7 2021"
- board text removed: "niubit PiConsole v6 2021"
Changed lines of the file:
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@@
     (thickness 1.6)
     (drawings 26)
-    (tracks 240)
+    (tracks 242)
     (zones 0)
     (modules 28)
@@
     (effects (font (size 1 1) (thickness 0.15)))
   )
-  (gr_text "niubit PiConsole v6 2021" (at 130.81 137.16) (layer F.SilkS)
+  (gr_text "niubit PiConsole v7 2021" (at 130.81 137.16) (layer F.SilkS)
     (effects (font (size 1.5 1.5) (thickness 0.3)))
   )
@@
   (segment (start 154.700988 62.625988) (end 155.575 63.5) (width 0.3) (layer F.Cu) (net 3))
   (segment (start 146.924012 62.625988) (end 154.700988 62.625988) (width 0.3) (layer F.Cu) (net 3))
-  (via (at 126.365 110.49) (size 0.8) (drill 0.4) (layers F.Cu B.Cu) (net 4))
-  (segment (start 126.365 101.6) (end 126.365 110.49) (width 0.3) (layer F.Cu) (net 4))
-  (via (at 140.335 120.015) (size 0.8) (drill 0.4) (layers F.Cu B.Cu) (net 4))
-  (segment (start 130.81 110.49) (end 140.335 120.015) (width 0.3) (layer B.Cu) (net 4))
-  (segment (start 126.365 110.49) (end 130.81 110.49) (width 0.3) (layer B.Cu) (net 4))
-  (segment (start 161.985001 67.370001) (end 158.115 63.5) (width 0.3) (layer F.Cu) (net 4))
-  (segment (start 161.985001 113.495001) (end 161.985001 67.370001) (width 0.3) (layer F.Cu) (net 4))
-  (segment (start 141.732 121.412) (end 154.068002 121.412) (width 0.3) (layer F.Cu) (net 4))
-  (segment (start 154.068002 121.412) (end 161.985001 113.495001) (width 0.3) (layer F.Cu) (net 4))
-  (segment (start 140.335 120.015) (end 141.732 121.412) (width 0.3) (layer F.Cu) (net 4))
+  (via (at 130.31 105.885) (size 0.8) (drill 0.4) (layers F.Cu B.Cu) (net 4))
+  (segment (start 130.31 105.545) (end 130.31 105.885) (width 0.3) (layer B.Cu) (net 4))
+  (segment (start 126.365 101.6) (end 130.31 105.545) (width 0.3) (layer B.Cu) (net 4))
+  (segment (start 162.81 68.195) (end 158.115 63.5) (width 0.3) (layer F.Cu) (net 4))
+  (segment (start 156.31 104.385) (end 162.81 97.885) (width 0.3) (layer F.Cu) (net 4))
+  (segment (start 147.87334 104.385) (end 156.31 104.385) (width 0.3) (layer F.Cu) (net 4))
+  (segment (start 143.793339 108.465001) (end 147.87334 104.385) (width 0.3) (layer F.Cu) (net 4))
+  (segment (start 162.81 97.885) (end 162.81 68.195) (width 0.3) (layer F.Cu) (net 4))
+  (segment (start 131.459 108.465001) (end 143.793339 108.465001) (width 0.3) (layer F.Cu) (net 4))
+  (segment (start 130.31 107.316001) (end 131.459 108.465001) (width 0.3) (layer F.Cu) (net 4))
+  (segment (start 130.31 105.885) (end 130.31 107.316001) (width 0.3) (layer F.Cu) (net 4))
   (segment (start 153.67 73.66) (end 155.575 71.755) (width 0.3) (layer F.Cu) (net 5))
   (segment (start 149.225 73.66) (end 153.67 73.66) (width 0.3) (layer F.Cu) (net 5))
@@
   (segment (start 141.605 115.137998) (end 129.337002 102.87) (width 0.3) (layer B.Cu) (net 39))
   (segment (start 141.605 128.905) (end 141.605 115.137998) (width 0.3) (layer B.Cu) (net 39))
-  (via (at 127.889 104.14) (size 0.8) (drill 0.4) (layers F.Cu B.Cu) (net 41))
+  (segment (start 127.635 128.27) (end 134.135 128.27) (width 0.3) (layer F.Cu) (net 41))
   (segment (start 123.825 102.235) (end 123.825 101.6) (width 0.3) (layer B.Cu) (net 41))
-  (segment (start 125.73 104.14) (end 123.825 102.235) (width 0.3) (layer B.Cu) (net 41))
-  (segment (start 127.889 104.14) (end 125.73 104.14) (width 0.3) (layer B.Cu) (net 41))
-  (segment (start 127 128.27) (end 127.635 128.27) (width 0.3) (layer F.Cu) (net 41))
-  (segment (start 126.000001 127.270001) (end 127 128.27) (width 0.3) (layer F.Cu) (net 41))
+  (via (at 127.889 105.885) (size 0.8) (drill 0.4) (layers F.Cu B.Cu) (net 41))
   (segment (start 127.889 112.21312) (end 126.000001 114.102119) (width 0.3) (layer F.Cu) (net 41))
   (segment (start 126.000001 114.102119) (end 126.000001 127.270001) (width 0.3) (layer F.Cu) (net 41))
-  (segment (start 127.889 104.14) (end 127.889 112.21312) (width 0.3) (layer F.Cu) (net 41))
-  (segment (start 127.635 128.27) (end 134.135 128.27) (width 0.3) (layer F.Cu) (net 41))
+  (segment (start 126.000001 127.270001) (end 127 128.27) (width 0.3) (layer F.Cu) (net 41))
+  (segment (start 127 128.27) (end 127.635 128.27) (width 0.3) (layer F.Cu) (net 41))
+  (segment (start 123.825 101.6) (end 123.825 102.9) (width 0.3) (layer B.Cu) (net 41))
+  (segment (start 126.81 105.885) (end 127.889 105.885) (width 0.3) (layer B.Cu) (net 41))
+  (segment (start 123.825 102.9) (end 126.81 105.885) (width 0.3) (layer B.Cu) (net 41))
+  (segment (start 127.889 112.21312) (end 127.889 105.885) (width 0.3) (layer F.Cu) (net 41))
   (zone (net 2) (net_name GND) (layer F.Cu) (hatch edge 0.508)
     (connect_pads (clearance 0.508))
