File: pcb/piconsole.kicad_sch (KiCad schematic)
At the start: 25 parts, among them J1 Bat, J2 GPIO, SW1 Up, SW2 Down, SW3 Left, SW4 Right, SW5 A, SW6 B, SW7 SW_SPDT, SW8 RESET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

Commit message: Nueva v7 (aún no se había fabricado)
Parts:
- BZ1: footprint Buzzer_Beeper:Buzzer_12x9.5RM7.6 -> Buzzer_Beeper:MagneticBuzzer_ProSignal_ABT-410-RC
Changed lines of the file:
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@@
       (effects (font (size 1.27 1.27)) (justify left))
     )
-    (property "Footprint" "Buzzer_Beeper:Buzzer_12x9.5RM7.6" (id 2) (at 143.51 144.78 90)
+    (property "Footprint" "Buzzer_Beeper:MagneticBuzzer_ProSignal_ABT-410-RC" (id 2) (at 143.51 144.78 90)
       (effects (font (size 1.27 1.27)) hide)
     )
@@
     )
     (path "/00000000-0000-0000-0000-000060d25ad7"
-      (reference "BZ1") (unit 1) (value "Buzzer") (footprint "Buzzer_Beeper:Buzzer_12x9.5RM7.6")
+      (reference "BZ1") (unit 1) (value "Buzzer") (footprint "Buzzer_Beeper:MagneticBuzzer_ProSignal_ABT-410-RC")
     )
     (path "/00000000-0000-0000-0000-000060d27b37"
